Commit message: (roseus_bt) Fix tutorial SubTreePlus port remapping

File: roseus_bt/sample/models/t07_xacro.xml.xacro (robot description, xacro)
@@ -5,5 +5,5 @@
   <xacro:include filename="$(find roseus_bt)/sample/models/t07_xacro_sweep_task.xml.xacro"
                  ns="sweep_task"/>
-  <xacro:property name="namespace" value="/t07_xacro"/>
+  <xacro:property name="namespace" value="/t05_subtrees"/>
   <!-- ////////// -->
     <BehaviorTree ID="BehaviorTree">
@@ -12,5 +12,5 @@
             <Action ID="setCoords" name="setBottleCoords" coords="$${bottle_coords}"/>
             <Sequence>
-                <SubTreePlus ID="PourTask" coords="bottle_coords"/>
+                <SubTreePlus ID="PourTask" coords="$${bottle_coords}"/>
                 <SubTreePlus ID="SweepTask"/>
             </Sequence>

File: roseus_bt/sample/models/t07_xacro_sweep_task.xml.xacro (robot description, xacro)
@@ -9,7 +9,9 @@
                 <Action ID="MoveTo" spot="broom-front"/>
             </Fallback>
-            <Timeout msec="5000">
-                <Action ID="SweepFloor"/>
-            </Timeout>
+            <ForceSuccess>
+                <Timeout msec="5000">
+                    <Action ID="SweepFloor"/>
+                </Timeout>
+            </ForceSuccess>
         </Sequence>
     </BehaviorTree>
